Commit message: add Mujoco sim2sim validation

File: legged_gym/resources/robots/q1/q1_box.urdf (robot description, URDF)
Before this commit: robot Q1-V2.0-URDF-0526, 24 links, 23 joints
Links:
- link left_ankle_pitch_link: geometry collision box size=0.04 0.05 0.02; visual mesh filename=/root/autodl-tmp/assets/robots/Q1-V2.0-URDF-0526/meshes/lef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
- link left_elbow_link: geometry collision box size=0.16 0.05 0.05; visual mesh filename=/root/autodl-tmp/assets/robots/Q1-V2.0-URDF-0526/meshes/lef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
- link left_hip_yaw_link: geometry collision box size=0.09 0.09 0.07; visual mesh filename=/root/autodl-tmp/assets/robots/Q1-V2.0-URDF-0526/meshes/lef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
- link left_knee_link: geometry collision box size=0.08 0.09 0.12; visual mesh filename=/root/autodl-tmp/assets/robots/Q1-V2.0-URDF-0526/meshes/lef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
- link left_shoulder_yaw_link: geometry collision box size=0.07 0.05 0.05; visual mesh filename=/root/autodl-tmp/assets/robots/Q1-V2.0-URDF-0526/meshes/lef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
- link pelvis: geometry collision box size=0.10 0.10 0.065; visual mesh filename=/root/autodl-tmp/assets/robots/Q1-V2.0-URDF-0526/meshes/pel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
- link right_ankle_pitch_link: geometry collision box size=0.04 0.05 0.02; visual mesh filename=/root/autodl-tmp/assets/robots/Q1-V2.0-URDF-0526/meshes/rig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
- link right_elbow_link: geometry collision box size=0.16 0.05 0.05; visual mesh filename=/root/autodl-tmp/assets/robots/Q1-V2.0-URDF-0526/meshes/rig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
- link right_hip_yaw_link: geometry collision box size=0.09 0.09 0.07; visual mesh filename=/root/autodl-tmp/assets/robots/Q1-V2.0-URDF-0526/meshes/rig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
- link right_knee_link: geometry collision box size=0.08 0.09 0.12; visual mesh filename=/root/autodl-tmp/assets/robots/Q1-V2.0-URDF-0526/meshes/rig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
- link right_shoulder_yaw_link: geometry collision box size=0.07 0.05 0.05; visual mesh filename=/root/autodl-tmp/assets/robots/Q1-V2.0-URDF-0526/meshes/rig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

Commit message: add g1 mujoco validation

File: legged_gym/resources/robots/q1/q1_box.urdf (robot description, URDF)
Before this commit: robot Q1-V2.0-URDF-0526, 24 links, 23 joints
Links:
- link head_link: geometry collision box size=0.12 0.09 0.12; visual mesh filename=meshes/head_link.STL
- link left_ankle_pitch_link: geometry collision box size=0.00 0.00 0.00; visual mesh filename=meshes/left_ankle_pitch_link.STL
- link left_ankle_roll_link: geometry collision sphere radius=0.008; collision sphere radius=0.008
- link left_elbow_link: geometry collision box size=0.16 0.05 0.05; visual mesh filename=meshes/left_elbow_link.STL
- link left_hip_pitch_link: geometry collision box size=0.00 0.00 0.00; visual mesh filename=meshes/left_hip_pitch_link.STL
- link left_hip_roll_link: geometry collision box size=0.09 0.08 0.08; visual mesh filename=meshes/left_hip_roll_link.STL
- link left_hip_yaw_link: geometry collision box size=0.09 0.09 0.07; visual mesh filename=meshes/left_hip_yaw_link.STL
- link left_knee_link: geometry collision box size=0.08 0.09 0.12; visual mesh filename=meshes/left_knee_link.STL
- link left_shoulder_pitch_link: geometry collision box size=0.0 0.0 0.0; visual mesh filename=meshes/left_shoulder_pitch_link.STL
- link left_shoulder_roll_link: geometry collision box size=0.07 0.05 0.09; visual mesh filename=meshes/left_shoulder_roll_link.STL
- link left_shoulder_yaw_link: geometry collision box size=0.07 0.05 0.05; visual mesh filename=meshes/left_shoulder_yaw_link.STL
- link pelvis: geometry collision box size=0.10 0.10 0.065; visual mesh filename=meshes/pelvis.STL
- link right_ankle_pitch_link: geometry collision box size=0.00 0.00 0.00; visual mesh filename=meshes/right_ankle_pitch_link.STL
- link right_ankle_roll_link: geometry collision sphere radius=0.008; collision sphere radius=0.008
- link right_elbow_link: geometry collision box size=0.16 0.05 0.05; visual mesh filename=meshes/right_elbow_link.STL
- link right_hip_pitch_link: geometry collision box size=0.0 0.0 0.0; visual mesh filename=meshes/right_hip_pitch_link.STL
- link right_hip_roll_link: geometry collision box size=0.09 0.08 0.08; visual mesh filename=meshes/right_hip_roll_link.STL
- link right_hip_yaw_link: geometry collision box size=0.09 0.09 0.07; visual mesh filename=meshes/right_hip_yaw_link.STL
- link right_knee_link: geometry collision box size=0.08 0.09 0.12; visual mesh filename=meshes/right_knee_link.STL
- link right_shoulder_pitch_link: geometry collision box size=0.0 0.0 0.0; visual mesh filename=meshes/right_shoulder_pitch_link.STL
- link right_shoulder_roll_link: geometry collision box size=0.07 0.05 0.09; visual mesh filename=meshes/right_shoulder_roll_link.STL
- link right_shoulder_yaw_link: geometry collision box size=0.07 0.05 0.05; visual mesh filename=meshes/right_shoulder_yaw_link.STL
- link torso_link: geometry collision box size=0.16 0.14 0.20; visual mesh filename=meshes/torso_link.STL
- link waist_roll_link: geometry collision box size=0.10 0.12 0.06; visual mesh filename=meshes/waist_roll_link.STL
